File: ESC-power-epc.kicad_pcb (KiCad board)
At the start: 4 copper layers, 50 x 100 mm, 66 parts, among them Q1 EPC2302, Q2 EPC2302, Q3 EPC2302, Q4 EPC2302, Q5 EPC2302, Q6 EPC2302, U1 LM5113SD/NOPB, U2 LM5113SD/NOPB, U3 INA181A2, U4 INA181A2, U5 INA181A2, U6 LM5113SD/NOPB

Commit message: before changing connector
Parts:
- removed R37, R38: 2k2, Resistor_SMD:R_0805_2012Metric
- removed R49, R50, R51, R52, R53, R54: R, Resistor_SMD:R_0805_2012Metric
- added C1: 1u, Capacitor_SMD:C_0402_1005Metric, B.Cu at (77.0, 83.8)
- added C10: 100n/100V, Capacitor_SMD:C_0603_1608Metric, F.Cu at (72.2, 78.8)
- added C11: 100n/100V, Capacitor_SMD:C_0603_1608Metric, F.Cu at (72.2, 66.8)
- added C2: 1u, Capacitor_SMD:C_0805_2012Metric, F.Cu at (171.2, 82.0)
- added C25: 2.2u/100V, Capacitor_SMD:C_0805_2012Metric, F.Cu at (175.5, 62.5)
- added C26: 2.2u/100V, Capacitor_SMD:C_0805_2012Metric, F.Cu at (176.8, 66.9)
- added C27: 2.2u/100V, Capacitor_SMD:C_0805_2012Metric, F.Cu at (181.3, 66.9)
- added C28: 2.2u/100V, Capacitor_SMD:C_0805_2012Metric, F.Cu at (176.8, 75.9)
- added C29: 2.2u/100V, Capacitor_SMD:C_0805_2012Metric, F.Cu at (181.3, 69.9)
- added C3: 1u, Capacitor_SMD:C_0805_2012Metric, F.Cu at (175.7, 82.0)
- added C30: 2.2u/100V, Capacitor_SMD:C_0805_2012Metric, F.Cu at (176.8, 72.9)
- added C31: 2.2u/100V, Capacitor_SMD:C_0805_2012Metric, F.Cu at (185.8, 65.5)
- added C32: 1u, Capacitor_SMD:C_0805_2012Metric, F.Cu at (108.2, 120.8)
- added C33: 100n, Capacitor_SMD:C_0805_2012Metric, F.Cu at (100.8, 110.0)
- added C34: 1n, Capacitor_SMD:C_0805_2012Metric, F.Cu at (101.0, 122.8)
- added C35: 1u, Capacitor_SMD:C_0805_2012Metric, F.Cu at (93.5, 119.5)
- added C36: 100n/100V, Capacitor_SMD:C_0603_1608Metric, F.Cu at (118.0, 66.8)
- added C37: 100n/100V, Capacitor_SMD:C_0603_1608Metric, F.Cu at (118.0, 68.2)
- added C38: 2.2u/100V, Capacitor_SMD:C_0805_2012Metric, F.Cu at (144.4, 89.5)
- added C39: 2.2u/100V, Capacitor_SMD:C_0805_2012Metric, F.Cu at (149.6, 82.0)
- added C4: 100n/100V, Capacitor_SMD:C_0603_1608Metric, F.Cu at (72.2, 69.8)
- added C41: 2.2u/100V, Capacitor_SMD:C_0805_2012Metric, F.Cu at (148.9, 86.5)
- added C42: 2.2u/100V, Capacitor_SMD:C_0805_2012Metric, F.Cu at (157.8, 85.0)
- added C43: 2.2u/100V, Capacitor_SMD:C_0805_2012Metric, F.Cu at (153.3, 85.0)
- added C44: 2.2u/100V, Capacitor_SMD:C_0805_2012Metric, F.Cu at (148.9, 89.5)
- added C45: 2.2u/100V, Capacitor_SMD:C_0805_2012Metric, F.Cu at (158.5, 82.0)
- added C46: 100n/100V, Capacitor_SMD:C_0603_1608Metric, F.Cu at (118.0, 69.8)
- added C47: 100n/100V, Capacitor_SMD:C_0603_1608Metric, F.Cu at (118.0, 71.2)
- added C48: 100n/100V, Capacitor_SMD:C_0603_1608Metric, F.Cu at (118.0, 72.8)
- added C49: 100n/100V, Capacitor_SMD:C_0603_1608Metric, F.Cu at (118.0, 74.2)
- added C5: 100n/100V, Capacitor_SMD:C_0603_1608Metric, F.Cu at (72.2, 71.2)
- added C50: 100n/100V, Capacitor_SMD:C_0603_1608Metric, F.Cu at (118.0, 75.8)
- added C56: 2.2u/100V, Capacitor_SMD:C_0805_2012Metric, F.Cu at (148.9, 66.9)
- added C57: 2.2u/100V, Capacitor_SMD:C_0805_2012Metric, F.Cu at (144.4, 75.9)
- added C58: 2.2u/100V, Capacitor_SMD:C_0805_2012Metric, F.Cu at (148.9, 69.9)
- added C59: 2.2u/100V, Capacitor_SMD:C_0805_2012Metric, F.Cu at (144.4, 72.9)
- added C6: 100n/100V, Capacitor_SMD:C_0603_1608Metric, F.Cu at (72.2, 72.8)
- added C60: 2.2u/100V, Capacitor_SMD:C_0805_2012Metric, F.Cu at (153.3, 65.5)
- added C61: 1u, Capacitor_SMD:C_0805_2012Metric, F.Cu at (124.2, 124.5)
- added C62: 1u, Capacitor_SMD:C_0402_1005Metric, F.Cu at (78.8, 80.5)
- added C63: 1u, Capacitor_SMD:C_0402_1005Metric, F.Cu at (103.2, 81.0)
- added C64: 1u, Capacitor_SMD:C_0402_1005Metric, F.Cu at (124.0, 81.0)
- added C65: 100n, Capacitor_SMD:C_0805_2012Metric, F.Cu at (117.5, 107.0)
- added C66: 1n, Capacitor_SMD:C_0805_2012Metric, F.Cu at (117.5, 121.8)
- added C7: 100n/100V, Capacitor_SMD:C_0603_1608Metric, F.Cu at (72.2, 74.2)
- added C8: 100n/100V, Capacitor_SMD:C_0603_1608Metric, F.Cu at (72.2, 75.8)
- added C9: 100n/100V, Capacitor_SMD:C_0603_1608Metric, F.Cu at (72.2, 77.2)
- added J1: GATE, Connector_PinHeader_2.54mm:PinHeader_2x04_P2.54mm_Vertical, F.Cu at (101.7, 95.3)
- added J2: Conn_01x02, Connector_PinHeader_2.54mm:PinHeader_1x02_P2.54mm_Vertical, F.Cu at (124.2, 92.8)
- added J3: Conn_01x04, Connector_PinHeader_2.54mm:PinHeader_2x02_P2.54mm_Vertical, F.Cu at (92.5, 129.0)
- added J4: GATE, Connector_PinHeader_2.54mm:PinHeader_2x04_P2.54mm_Vertical, F.Cu at (113.7, 132.0)
- added NT10: NetTie_2, NetTie:NetTie-2_SMD_Pad0.5mm, F.Cu at (52.8, 82.2)
- added NT11: NetTie_2, NetTie:NetTie-2_SMD_Pad0.5mm, F.Cu at (63.5, 97.5)
- added NT12: NetTie_2, NetTie:NetTie-2_SMD_Pad0.5mm, F.Cu at (48.3, 85.8)
- added NT7: NetTie_2, NetTie:NetTie-2_SMD_Pad0.5mm, F.Cu at (56.8, 88.7)
- added NT8: NetTie_2, NetTie:NetTie-2_SMD_Pad0.5mm, F.Cu at (52.8, 91.2)
- added NT9: NetTie_2, NetTie:NetTie-2_SMD_Pad0.5mm, F.Cu at (56.8, 79.7)
- added R1: R, Resistor_SMD:R_0402_1005Metric, F.Cu at (76.7, 79.0)
- added R14: R, Resistor_SMD:R_0402_1005Metric, F.Cu at (100.0, 78.8)
- added R15: R, Resistor_SMD:R_0402_1005Metric, F.Cu at (101.0, 78.8)
- added R16: R, Resistor_SMD:R_0402_1005Metric, F.Cu at (106.2, 78.5)
- added R17: R, Resistor_SMD:R_0402_1005Metric, F.Cu at (105.2, 78.5)
- added R18: R, Resistor_SMD:R_0402_1005Metric, F.Cu at (122.5, 79.2)
- added R19: R, Resistor_SMD:R_0402_1005Metric, F.Cu at (121.5, 79.2)
- added R2: R, Resistor_SMD:R_0402_1005Metric, F.Cu at (75.7, 79.0)
- added R20: R, Resistor_SMD:R_0402_1005Metric, F.Cu at (127.2, 79.2)
- added R21: R, Resistor_SMD:R_0402_1005Metric, F.Cu at (128.2, 79.2)
- added R22: 39k, Resistor_SMD:R_0805_2012Metric, F.Cu at (86.7, 134.8)
- added R23: 1k, Resistor_SMD:R_0805_2012Metric, F.Cu at (101.0, 119.0)
- added R24: 2k2, Resistor_SMD:R_0805_2012Metric, F.Cu at (105.5, 129.8)
- added R25: R, Resistor_SMD:R_2512_6332Metric, F.Cu at (80.0, 63.5)
- added R27: R, Resistor_SMD:R_2512_6332Metric, F.Cu at (125.2, 62.5)
- added R28: 3m, Froste:0805W, F.Cu at (132.8, 67.5)
- added R3: R, Resistor_SMD:R_0402_1005Metric, F.Cu at (81.5, 79.0)
- added R30: 3m, Froste:0805W, F.Cu at (132.8, 73.5)
- added R31: 3m, Froste:0805W, F.Cu at (132.8, 76.5)
- added R4: R, Resistor_SMD:R_0402_1005Metric, F.Cu at (82.5, 79.0)
- added U7: INA240A1D, Package_SO:SOIC-8_3.9x4.9mm_P1.27mm, F.Cu at (108.0, 114.0)
- added U8: INA240A1D, Package_SO:SOIC-8_3.9x4.9mm_P1.27mm, F.Cu at (93.0, 114.0)
- added U9: INA181A2, Package_TO_SOT_SMD:SOT-23-6, F.Cu at (117.5, 113.8)
- C12: value 680uF 63V -> 100n/100V; footprint Capacitor_THT:CP_Radial_D10.0mm_P5.00mm -> Capacitor_SMD:C_0603_1608Metric
- C14, C15, C18, C19, C22, C23: value 2.2u/100V -> 100n/100V; footprint Capacitor_SMD:C_1210_3225Metric -> Capacitor_SMD:C_0603_1608Metric
- C17, C21: value 100n -> 100n/100V; footprint Capacitor_SMD:C_0805_2012Metric -> Capacitor_SMD:C_0603_1608Metric
- C20: value 1n -> 100n/100V; footprint Capacitor_SMD:C_0805_2012Metric -> Capacitor_SMD:C_0603_1608Metric
- C24: value 1n -> 2.2u/100V
- C40, C53, C54, C55: value C -> 2.2u/100V
- C51, C52: value C -> 100n/100V; footprint Capacitor_SMD:C_0805_2012Metric -> Capacitor_SMD:C_0603_1608Metric
- Q1, Q2, Q3, Q4, Q5, Q6: footprint epc2:EPC2302 -> epc:EPC2302
- R10, R13, R7: value 0.5mOhm -> 3m; footprint Resistor_SMD:R_2512_6332Metric -> Froste:0805W
- R11, R12, R5, R6, R8: value 10 -> 3m; footprint Resistor_SMD:R_0805_2012Metric -> Froste:0805W
- R29: value 1k -> 3m; footprint Resistor_SMD:R_0805_2012Metric -> Froste:0805W
- R32: value 1k -> 39k
- R34: value 39k -> 1k
- R35: value 39k -> 2k2
- R9: value 10 -> R; footprint Resistor_SMD:R_0805_2012Metric -> Resistor_SMD:R_2512_6332Metric
- U1, U2, U6: footprint lm5113:LM5113SD&slash_NOPB -> lm5113:LM5113SD_NOPB
- U4: value INA181A2 -> INA240A1D; footprint Package_TO_SOT_SMD:SOT-23-6 -> Package_SO:SOIC-8_3.9x4.9mm_P1.27mm
- moved NT1 103.5 mm to (43.9, 99.8)
- moved NT4 93.0 mm to (60.0, 83.8)
- moved R32 90.6 mm to (99.8, 134.8)
- moved R33 84.4 mm to (86.7, 130.2)
- moved C13 80.8 mm to (84.5, 109.8)
- moved R36 80.2 mm to (106.2, 134.5)
- moved U3 80.0 mm to (85.0, 114.5)
- moved R34 78.2 mm to (117.5, 118.2)
- moved C16 75.3 mm to (85.0, 123.0)
- moved H1 69.2 mm to (72.0, 97.2), turned to 180 degrees
- moved H2 64.9 mm to (72.2, 106.8)
- moved C14 59.0 mm to (72.2, 68.2), turned to 180 degrees
- moved R26 58.8 mm to (84.8, 119.0)
- moved R35 56.3 mm to (100.0, 130.2)
- moved U4 52.7 mm to (124.2, 114.0)
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Connections:
- net /MOSFETS/CURR_A renamed /CURRENT_A
- net /MOSFETS/SA_N renamed /GaN_A/SA_N
- net /MOSFETS/SA_P renamed /GaN_A/SA_P
- net /MOSFETS/SC_N renamed /GaN_B/SA_N
- net /MOSFETS/SC_P renamed /GaN_B/SA_P
- net /MOSFETS/SENSE_A renamed /SENSE_A
- C17 pad 1: +3V3 -> V_SUPPLY
- C20 pad 1: /MOSFETS/CURR_B -> V_SUPPLY
- C21 pad 1: +3V3 -> V_SUPPLY
- C24 pad 1: /MOSFETS/CURR_C -> V_SUPPLY
- C40 pad 1: Net-(C40-Pad1) -> V_SUPPLY
- C40 pad 2: /MOSFETS/VSA -> GND
- C51 pad 1: Net-(C51-Pad1) -> V_SUPPLY
- C52 pad 1: Net-(C52-Pad1) -> V_SUPPLY
- C52 pad 2: /MOSFETS/VSB -> GND
- C53 pad 1: Net-(C53-Pad1) -> V_SUPPLY
- C54 pad 1: Net-(C54-Pad1) -> V_SUPPLY
- C54 pad 2: /MOSFETS/VSC -> GND
- C55 pad 1: Net-(C55-Pad1) -> V_SUPPLY
- H3 pad 1: /MOSFETS/VSA -> /GATE/VSA
- H4 pad 1: /MOSFETS/VSB -> /GATE/VSB
- H5 pad 1: /MOSFETS/VSC -> /GATE/VSC
- NT3 pad 1: /MOSFETS/SB_P -> /GATE/VSB
- NT4 pad 1: /MOSFETS/SB_N -> Net-(NT4-Pad1)
- NT4 pad 2: GND -> Net-(NT4-Pad2)
- Q1 pad 1: Net-(Q1-Pad1) -> /GATE/GH_A
- Q1 pad 2: /MOSFETS/VSA -> Net-(NT8-Pad2)
- Q1 pad 4: /MOSFETS/VSA -> Net-(NT8-Pad2)
- Q1 pad 6: /MOSFETS/VSA -> Net-(NT8-Pad2)
- Q2 pad 1: Net-(Q2-Pad1) -> /GATE/GH_B
- Q2 pad 2: /MOSFETS/VSB -> Net-(NT4-Pad2)
- Q2 pad 4: /MOSFETS/VSB -> Net-(NT4-Pad2)
- Q2 pad 6: /MOSFETS/VSB -> Net-(NT4-Pad2)
- Q3 pad 1: Net-(Q3-Pad1) -> /GATE/GL_B
- Q3 pad 2: /MOSFETS/VSC -> Net-(NT5-Pad2)
- Q3 pad 3: V_SUPPLY -> Net-(NT4-Pad2)
- Q3 pad 4: /MOSFETS/VSC -> Net-(NT5-Pad2)
- Q3 pad 5: V_SUPPLY -> Net-(NT4-Pad2)
- Q3 pad 6: /MOSFETS/VSC -> Net-(NT5-Pad2)
- Q3 pad 7: V_SUPPLY -> Net-(NT4-Pad2)
- Q4 pad 1: Net-(Q4-Pad1) -> /GATE/GL_A
- Q4 pad 3: /MOSFETS/VSA -> Net-(NT8-Pad2)
- Q4 pad 5: /MOSFETS/VSA -> Net-(NT8-Pad2)
- Q4 pad 7: /MOSFETS/VSA -> Net-(NT8-Pad2)
- Q5 pad 1: Net-(Q5-Pad1) -> /GATE/GH_C
- Q5 pad 2: Net-(NT3-Pad2) -> Net-(NT10-Pad2)
- Q5 pad 3: /MOSFETS/VSB -> V_SUPPLY
- Q5 pad 4: Net-(NT3-Pad2) -> Net-(NT10-Pad2)
- Q5 pad 5: /MOSFETS/VSB -> V_SUPPLY
- Q5 pad 6: Net-(NT3-Pad2) -> Net-(NT10-Pad2)
- Q5 pad 7: /MOSFETS/VSB -> V_SUPPLY
- Q6 pad 1: Net-(Q6-Pad1) -> /GATE/GL_C
- Q6 pad 2: Net-(NT5-Pad2) -> Net-(NT11-Pad2)
- Q6 pad 3: /MOSFETS/VSC -> Net-(NT10-Pad2)
- Q6 pad 4: Net-(NT5-Pad2) -> Net-(NT11-Pad2)
- Q6 pad 5: /MOSFETS/VSC -> Net-(NT10-Pad2)
- Q6 pad 6: Net-(NT5-Pad2) -> Net-(NT11-Pad2)
- Q6 pad 7: /MOSFETS/VSC -> Net-(NT10-Pad2)
- R10 pad 1: Net-(NT3-Pad2) -> Net-(NT5-Pad2)
- R11 pad 1: /MOSFETS/GH_C -> Net-(NT5-Pad2)
- R11 pad 2: Net-(Q3-Pad1) -> GND
- R12 pad 1: /MOSFETS/GL_C -> Net-(NT5-Pad2)
- R12 pad 2: Net-(Q6-Pad1) -> GND
- R29 pad 1: Net-(R29-Pad1) -> Net-(NT11-Pad2)
- R29 pad 2: /MOSFETS/CURR_B -> GND
- R32 pad 1: Net-(R32-Pad1) -> /GATE/VSC
- R32 pad 2: /MOSFETS/CURR_C -> /SENSE_C
- R33 pad 1: /MOSFETS/VSA -> /GATE/VSA
- R34 pad 1: /MOSFETS/VSB -> Net-(R34-Pad1)
- R34 pad 2: /MOSFETS/SENSE_B -> /CURRENT_C
- R35 pad 1: /MOSFETS/VSC -> GND
- R35 pad 2: /MOSFETS/SENSE_C -> /SENSE_C
- R5 pad 1: /MOSFETS/GH_A -> Net-(NT1-Pad2)
- R5 pad 2: Net-(Q1-Pad1) -> GND
- R6 pad 1: /MOSFETS/GL_A -> Net-(NT1-Pad2)
- R6 pad 2: Net-(Q4-Pad1) -> GND
- R8 pad 1: /MOSFETS/GH_B -> Net-(NT1-Pad2)
- R8 pad 2: Net-(Q2-Pad1) -> GND
- R9 pad 1: /MOSFETS/GL_B -> Net-(NT4-Pad2)
- R9 pad 2: Net-(Q5-Pad1) -> /GATE/VSB
- U1 pad 1: unconnected-(U1-Pad1) -> +5V
- U1 pad 10: unconnected-(U1-Pad10) -> Net-(R3-Pad1)
- U1 pad 11: unconnected-(U1-Pad11) -> GND
- U1 pad 2: unconnected-(U1-Pad2) -> Net-(C1-Pad2)
- U1 pad 3: unconnected-(U1-Pad3) -> Net-(R1-Pad1)
- U1 pad 4: unconnected-(U1-Pad4) -> Net-(R2-Pad1)
- U1 pad 5: unconnected-(U1-Pad5) -> /GATE/VSA
- U1 pad 6: unconnected-(U1-Pad6) -> /GATE/H1
- U1 pad 7: unconnected-(U1-Pad7) -> /GATE/L1
- U1 pad 8: unconnected-(U1-Pad8) -> GND
- U1 pad 9: unconnected-(U1-Pad9) -> Net-(R4-Pad1)
- U2 pad 1: unconnected-(U2-Pad1) -> +5V
- U2 pad 10: unconnected-(U2-Pad10) -> Net-(R16-Pad1)
- U2 pad 11: unconnected-(U2-Pad11) -> GND
- U2 pad 2: unconnected-(U2-Pad2) -> Net-(C2-Pad2)
- U2 pad 3: unconnected-(U2-Pad3) -> Net-(R14-Pad1)
- U2 pad 4: unconnected-(U2-Pad4) -> Net-(R15-Pad1)
- U2 pad 5: unconnected-(U2-Pad5) -> /GATE/VSB
- U2 pad 6: unconnected-(U2-Pad6) -> /GATE/H2
- U2 pad 7: unconnected-(U2-Pad7) -> /GATE/L2
- U2 pad 8: unconnected-(U2-Pad8) -> GND
- U2 pad 9: unconnected-(U2-Pad9) -> Net-(R17-Pad1)
- U4 pad 1: Net-(R29-Pad1) -> Net-(NT3-Pad2)
- U4 pad 2: GND -> Net-(U4-Pad2)
- U4 pad 3: /MOSFETS/SB_P -> unconnected-(U4-Pad3)
- U4 pad 4: /MOSFETS/SB_N -> Net-(U4-Pad2)
- U4 pad 5: +1V5 -> GND
- U5 pad 1: Net-(R32-Pad1) -> Net-(R23-Pad1)
- U6 pad 1: unconnected-(U6-Pad1) -> +5V
- U6 pad 10: unconnected-(U6-Pad10) -> Net-(R20-Pad1)
- U6 pad 11: unconnected-(U6-Pad11) -> GND
- U6 pad 2: unconnected-(U6-Pad2) -> Net-(C3-Pad2)
- U6 pad 3: unconnected-(U6-Pad3) -> Net-(R18-Pad1)
- U6 pad 4: unconnected-(U6-Pad4) -> Net-(R19-Pad1)
- U6 pad 5: unconnected-(U6-Pad5) -> /GATE/VSC
- U6 pad 6: unconnected-(U6-Pad6) -> /GATE/H3
- U6 pad 7: unconnected-(U6-Pad7) -> /GATE/L3
- U6 pad 8: unconnected-(U6-Pad8) -> GND
- U6 pad 9: unconnected-(U6-Pad9) -> Net-(R21-Pad1)
Routing:
- net (no net): track 213.5 -> 0.00 mm
Other:
- board size 50 x 100 mm -> 70 x 90 mm

Commit message: before meeting
Parts:
- moved R27 48.5 mm to (76.8, 63.5)
- moved C36 48.4 mm to (69.7, 67.8)
- moved C37 48.4 mm to (69.7, 69.2)
- moved C46 48.4 mm to (69.7, 70.8)
- moved C47 48.4 mm to (69.7, 72.2)
- moved C48 48.4 mm to (69.7, 73.8)
- moved C49 48.4 mm to (69.7, 75.2)
- moved C50 48.4 mm to (69.6, 76.8)
- moved C51 48.4 mm to (69.7, 78.2)
- moved C52 48.4 mm to (69.7, 79.8)
- moved Q6 48.4 mm to (79.4, 74.7)
- moved R28 48.4 mm to (84.4, 68.5)
- moved R29 48.4 mm to (84.4, 71.5)
- moved R30 48.4 mm to (84.4, 74.5)
- moved R31 48.4 mm to (84.4, 77.5)
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Connections:
- J1 pad 1: /GATE/H1 -> /GATE/H3
- J1 pad 2: GND -> /GATE/H2
- J1 pad 3: /GATE/H2 -> GND
- J1 pad 4: /GATE/H3 -> /GATE/H1
- J1 pad 5: /GATE/L1 -> /GATE/L3
- J1 pad 7: /GATE/L3 -> +5V
- J1 pad 8: +12V -> /GATE/L1
- J4 pad 1: +5V -> +3V3
- J4 pad 2: +3V3 -> GND
- J4 pad 6: unconnected-(J4-Pad6) -> /TEMP_MOSFET
- J4 pad 8: GND -> +12V
Routing:
- net Net-(NT10-Pad2): track 0.00 -> 11.2 mm, vias 0 -> 6
- net V_SUPPLY: track 0.00 -> 10.2 mm, vias 0 -> 6
- net Net-(R19-Pad1): track 0.00 -> 6.55 mm
- net Net-(R18-Pad1): track 0.00 -> 5.52 mm
- net Net-(R21-Pad1): track 0.00 -> 4.93 mm
- net Net-(NT11-Pad2): track 0.00 -> 3.74 mm, vias 0 -> 8
- net Net-(R20-Pad1): track 0.00 -> 3.14 mm
- net /GATE/GH_C: track 0.00 -> 3.02 mm
- net /GATE/GL_C: track 0.00 -> 2.64 mm
- net (no net): vias 0 -> 12
- added copper zone on F.Cu, net Net-(NT10-Pad2)
- added copper zone on F.Cu, net Net-(NT11-Pad2)
- added copper zone on F.Cu, net V_SUPPLY
Other:
- board size 70 x 90 mm -> 67 x 90 mm

Commit message: v0.1
Parts:
- added C67: 10u/100V, Capacitor_SMD:C_2220_5650Metric, F.Cu at (89.0, 45.3)
- added C69: 10u/100V, Capacitor_SMD:C_2220_5650Metric, F.Cu at (95.0, 45.3)
- added C75: 660u, Capacitor_THT:CP_Radial_D12.5mm_P5.00mm, F.Cu at (112.3, 49.4)
- added C76: 2u2, Capacitor_SMD:C_0805_2012Metric, F.Cu at (110.8, 128.8)
- added C77: 2u2, Capacitor_SMD:C_0805_2012Metric, F.Cu at (69.5, 113.2)
- added C78: 2u2, Capacitor_SMD:C_0805_2012Metric, F.Cu at (81.2, 113.2)
- added C79: 2u2, Capacitor_SMD:C_0805_2012Metric, F.Cu at (94.8, 113.2)
- added H10: MountingHole, MountingHole:MountingHole_3.2mm_M3, F.Cu at (69.2, 99.0)
- added H11: MountingHole, MountingHole:MountingHole_3.2mm_M3, F.Cu at (122.2, 100.0)
- added H6: MountingHole, MountingHole:MountingHole_3.2mm_M3, F.Cu at (69.2, 136.5)
- added H7: MountingHole, MountingHole:MountingHole_3.2mm_M3, F.Cu at (122.2, 136.5)
- added H8: MountingHole, MountingHole:MountingHole_3.2mm_M3, F.Cu at (102.8, 43.5)
- added H9: MountingHole, MountingHole:MountingHole_3.2mm_M3, F.Cu at (69.2, 43.5)
- added JP1: Jumper_3_Bridged12, Jumper:SolderJumper-3_P1.3mm_Open_RoundedPad1.0x1.5mm, F.Cu at (82.8, 127.0)
- added JP2: Jumper_3_Bridged12, Jumper:SolderJumper-3_P1.3mm_Open_RoundedPad1.0x1.5mm, F.Cu at (88.5, 127.0)
- added JP3: Jumper_3_Bridged12, Jumper:SolderJumper-3_P1.3mm_Open_RoundedPad1.0x1.5mm, F.Cu at (69.8, 127.0)
- added Q10: BSS138, Package_TO_SOT_SMD:SOT-23, F.Cu at (82.2, 89.2)
- added Q11: BSS138, Package_TO_SOT_SMD:SOT-23, F.Cu at (99.0, 85.0)
- added Q12: BSS138, Package_TO_SOT_SMD:SOT-23, F.Cu at (99.0, 88.5)
- added Q7: BSS138, Package_TO_SOT_SMD:SOT-23, F.Cu at (118.5, 89.2)
- added Q8: BSS138, Package_TO_SOT_SMD:SOT-23, F.Cu at (78.8, 89.2)
- added Q9: BSS138, Package_TO_SOT_SMD:SOT-23, F.Cu at (122.0, 89.2)
- added R37: 10k, Resistor_SMD:R_0805_2012Metric, F.Cu at (118.5, 86.2)
- added R38: 10k, Resistor_SMD:R_0805_2012Metric, F.Cu at (78.8, 92.2)
- added R39: 10k, Resistor_SMD:R_0805_2012Metric, F.Cu at (78.8, 86.2)
- added R40: 10k, Resistor_SMD:R_0805_2012Metric, F.Cu at (122.0, 92.2)
- added R41: 10k, Resistor_SMD:R_0805_2012Metric, F.Cu at (122.0, 86.2)
- added R42: 10k, Resistor_SMD:R_0805_2012Metric, F.Cu at (82.2, 92.2)
- added R43: 10k, Resistor_SMD:R_0805_2012Metric, F.Cu at (82.2, 86.2)
- added R44: 10k, Resistor_SMD:R_0805_2012Metric, F.Cu at (96.0, 85.0)
- added R45: 10k, Resistor_SMD:R_0805_2012Metric, F.Cu at (102.0, 85.0)
- added R46: 10k, Resistor_SMD:R_0805_2012Metric, F.Cu at (96.0, 88.5)
- added R47: 10k, Resistor_SMD:R_0805_2012Metric, F.Cu at (102.0, 88.5)
- added R48: NTC 10k, Resistor_SMD:R_0603_1608Metric, F.Cu at (75.8, 74.0)
- added R49: 10k, Resistor_SMD:R_0805_2012Metric, F.Cu at (110.8, 130.8)
- added R50: 1m, Resistor_SMD:R_2512_6332Metric, F.Cu at (97.5, 62.0)
- added R52: 1m, Resistor_SMD:R_2512_6332Metric, F.Cu at (117.2, 62.0)
- added R54: 1m, Resistor_SMD:R_2512_6332Metric, F.Cu at (78.0, 62.0)
- added TP1: GND, TestPoint:TestPoint_THTPad_D1.5mm_Drill0.7mm, F.Cu at (85.3, 56.8)
- added TP2: GND, TestPoint:TestPoint_THTPad_D1.5mm_Drill0.7mm, F.Cu at (83.3, 80.3)
- C1: footprint Capacitor_SMD:C_0402_1005Metric -> Capacitor_SMD:C_0805_2012Metric
- C2, C24, C25, C26, C27, C28, C29, C3, C30, C31, C38, C39, C40, C41, C42, C43, C44, C45, C53, C54, C55, C56, C57, C58, C59, C60: moved to B.Cu
- C32: value 1u -> 10u
- C35, C61: value 1u -> 10u/100V; footprint Capacitor_SMD:C_0805_2012Metric -> Capacitor_SMD:C_2220_5650Metric
- C62, C63, C64: footprint Capacitor_SMD:C_0402_1005Metric -> Capacitor_SMD:C_0603_1608Metric
- NT1, NT11, NT12, NT2, NT5, NT6: footprint NetTie:NetTie-2_SMD_Pad0.5mm -> Froste:NetTie-2_SMD_Pad0.26mm
- R1, R14, R15, R16, R17, R18, R19, R2, R20, R21, R3, R4: value R -> 10; footprint Resistor_SMD:R_0402_1005Metric -> Resistor_SMD:R_0603_1608Metric
- R10, R11, R12, R13, R28, R29, R30, R31, R5, R6, R7, R8: value 3m -> 2m
- R25, R27, R9: value R -> 10k; footprint Resistor_SMD:R_2512_6332Metric -> Resistor_SMD:R_0805_2012Metric
- U4, U7, U8: value INA240A1D -> AD8418; footprint Package_SO:SOIC-8_3.9x4.9mm_P1.27mm -> Package_SO:MSOP-8_3x3mm_P0.65mm
- moved C61 84.0 mm to (83.0, 45.3), turned to 90 degrees
- moved NT1 83.3 mm to (121.3, 68.9), turned to 180 degrees
- moved C3 79.6 mm to (75.2, 79.5), turned to 90 degrees
- moved NT2 78.7 mm to (122.7, 68.9)
- moved C60 78.5 mm to (70.7, 75.9), turned to 180 degrees
- moved H2 76.7 mm to (121.0, 44.5)
- moved C31 76.3 mm to (90.0, 76.0), turned to 180 degrees
- moved C54 74.3 mm to (70.7, 63.9), turned to 180 degrees
- moved C35 74.3 mm to (77.0, 45.3), turned to 90 degrees
- moved C56 73.6 mm to (70.7, 67.9), turned to 180 degrees
- moved C58 73.6 mm to (70.7, 71.9), turned to 180 degrees
- moved C29 70.7 mm to (90.0, 72.0), turned to 180 degrees
- moved C27 70.6 mm to (90.0, 68.0), turned to 180 degrees
- moved NT8 69.9 mm to (117.2, 64.2), turned to -90 degrees
- moved C53 69.8 mm to (70.7, 61.9), turned to 180 degrees
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Connections:
- net /GATE/GH_A renamed /GaN_A/GH
- net /GATE/GH_B renamed /GaN_B/GH
- net /GATE/GH_C renamed /GaN_C/GH
- net /GATE/GL_A renamed /GaN_A/GL
- net /GATE/GL_B renamed /GaN_B/GL
- net /GATE/GL_C renamed /GaN_C/GL
- net /GaN_A/SA_N renamed /GaN_A/S_N
- net /GaN_A/SA_P renamed /GaN_A/S_P
- net /GaN_B/SA_N renamed /GaN_B/S_N
- net /GaN_B/SA_P renamed /GaN_B/S_P
- net /GaN_C/SA_N renamed /GaN_C/S_N
- net /GaN_C/SA_P renamed /GaN_C/S_P
- net Net-(NT10-Pad1) renamed /GaN_C/IN+
- net Net-(NT4-Pad1) renamed /GaN_B/IN+
- net Net-(NT8-Pad1) renamed /GaN_A/IN+
- C1 pad 1: /GATE/VSA -> /VSA
- C16 pad 1: /CURRENT_A -> /GaN_A/CUR_SHUNT_LOW
- C2 pad 1: /GATE/VSB -> /VSB
- C3 pad 1: /GATE/VSC -> /VSC
- C32 pad 1: +3V3 -> 1V65
- C34 pad 1: /CURRENT_B -> /GaN_B/CUR_SHUNT_LOW
- C35 pad 1: +3V3 -> V_SUPPLY
- C61 pad 1: +3V3 -> V_SUPPLY
- C63 pad 1: unconnected-(C63-Pad1) -> +5V
- C66 pad 1: /CURRENT_C -> /GaN_C/CUR_SHUNT_LOW
- H3 pad 1: /GATE/VSA -> /VSA
- H4 pad 1: /GATE/VSB -> /VSB
- H5 pad 1: /GATE/VSC -> /VSC
- J1 pad 1: /GATE/H3 -> /Gate drivers/H3
- J1 pad 2: /GATE/H2 -> /Gate drivers/H2
- J1 pad 4: /GATE/H1 -> /Gate drivers/H1
- J1 pad 5: /GATE/L3 -> /Gate drivers/L3
- J1 pad 6: /GATE/L2 -> /Gate drivers/L2
- J1 pad 8: /GATE/L1 -> /Gate drivers/L1
- J4 pad 6: /TEMP_MOSFET -> /TEMP_FET
- NT3 pad 1: /GATE/VSB -> /GaN_B/IN-
- NT3 pad 2: Net-(NT3-Pad2) -> /VSB
- NT7 pad 1: /GATE/VSA -> /GaN_A/IN-
- NT7 pad 2: Net-(NT7-Pad2) -> /VSA
- NT9 pad 1: /GATE/VSC -> /GaN_C/IN-
- NT9 pad 2: Net-(NT9-Pad2) -> /VSC
- R22 pad 1: /GATE/VSB -> /VSB
- R23 pad 2: /CURRENT_B -> /GaN_B/CUR_SHUNT_LOW
- R25 pad 1: Net-(NT8-Pad2) -> 1V65
- R25 pad 2: /GATE/VSA -> GND
- R26 pad 2: /CURRENT_A -> /GaN_A/CUR_SHUNT_LOW
- R27 pad 1: Net-(NT10-Pad2) -> +3V3
- R27 pad 2: /GATE/VSC -> /Gate drivers/H1
- R32 pad 1: /GATE/VSC -> /VSC
- R33 pad 1: /GATE/VSA -> /VSA
- R34 pad 2: /CURRENT_C -> /GaN_C/CUR_SHUNT_LOW
- R9 pad 1: Net-(NT4-Pad2) -> +3V3
- R9 pad 2: /GATE/VSB -> 1V65
- U1 pad 5: /GATE/VSA -> /VSA
- U1 pad 6: /GATE/H1 -> Net-(Q7-Pad3)
- U1 pad 7: /GATE/L1 -> Net-(Q9-Pad3)
- U2 pad 5: /GATE/VSB -> /VSB
- U2 pad 6: /GATE/H2 -> Net-(Q11-Pad3)
- U2 pad 7: /GATE/L2 -> Net-(Q12-Pad3)
- U3 pad 5: +1V5 -> 1V65
- U4 pad 1: Net-(NT3-Pad2) -> /GaN_B/IN-
- U4 pad 2: Net-(U4-Pad2) -> GND
- U4 pad 3: unconnected-(U4-Pad3) -> GND
- U4 pad 4: Net-(U4-Pad2) -> unconnected-(U4-Pad4)
- U4 pad 5: GND -> /GaN_B/CUR_SHUNT_PHASE
- U4 pad 7: unconnected-(U4-Pad7) -> +3V3
- U5 pad 5: +1V5 -> 1V65
- U6 pad 5: /GATE/VSC -> /VSC
- U6 pad 6: /GATE/H3 -> Net-(Q8-Pad3)
- U6 pad 7: /GATE/L3 -> Net-(Q10-Pad3)
- U7 pad 1: Net-(NT7-Pad2) -> /GaN_A/IN-
- U7 pad 2: Net-(U7-Pad2) -> GND
- U7 pad 3: unconnected-(U7-Pad3) -> GND
- U7 pad 4: Net-(U7-Pad2) -> unconnected-(U7-Pad4)
- U7 pad 5: GND -> /GaN_A/CUR_SHUNT_PHASE
- U7 pad 7: unconnected-(U7-Pad7) -> +3V3
- U8 pad 1: Net-(NT9-Pad2) -> /GaN_C/IN-
- U8 pad 2: Net-(U8-Pad2) -> GND
- U8 pad 3: unconnected-(U8-Pad3) -> GND
- U8 pad 4: Net-(U8-Pad2) -> unconnected-(U8-Pad4)
- U8 pad 5: GND -> /GaN_C/CUR_SHUNT_PHASE
- U8 pad 7: unconnected-(U8-Pad7) -> +3V3
- U9 pad 5: +1V5 -> 1V65
Routing:
- net +3V3: track 0.00 -> 224.6 mm, vias 0 -> 14
- net /TEMP_FET: track 0.00 -> 116.8 mm, vias 0 -> 2
- net +5V: track 0.00 -> 106.3 mm, vias 0 -> 9
- net /VSC: track 0.00 -> 83.0 mm, vias 0 -> 2
- net /VSB: track 0.00 -> 80.3 mm, vias 0 -> 3
- net /GaN_A/S_N: track 0.00 -> 73.6 mm, vias 0 -> 2
- net /GaN_A/S_P: track 0.00 -> 72.2 mm, vias 0 -> 2
- net /GaN_A/IN-: track 0.00 -> 68.5 mm, vias 0 -> 2
- net /GaN_A/IN+: track 0.00 -> 67.5 mm, vias 0 -> 2
- net /GaN_B/S_N: track 0.00 -> 66.1 mm, vias 0 -> 2
- net /VSA: track 0.00 -> 65.5 mm, vias 0 -> 3
- net /GaN_B/S_P: track 0.00 -> 64.4 mm, vias 0 -> 2
- net /GaN_B/IN-: track 0.00 -> 64.2 mm, vias 0 -> 2
- net /GaN_B/IN+: track 0.00 -> 63.5 mm, vias 0 -> 2
- net /GaN_C/S_N: track 0.00 -> 60.1 mm, vias 0 -> 2
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- added copper zone on F.Cu, net /GaN_A/GH
- added copper zone on F.Cu, net /GaN_A/GL
- added copper zone on F.Cu, net /GaN_B/GH
- added copper zone on F.Cu, net /GaN_B/GL
- added copper zone on F.Cu, net /GaN_C/GH
- added copper zone on F.Cu, net /GaN_C/GL
- added copper zone on F.Cu, net /VSA
- added copper zone on F.Cu, net /VSB
- added copper zone on F.Cu, net /VSC
- added copper zone on B.Cu, net GND
- added copper zone on F.Cu, net GND
- added copper zone on In1.Cu, net GND
- added copper zone on In2.Cu, net GND
- added copper zone on F.Cu, net Net-(NT1-Pad2)
- added copper zone on F.Cu, net Net-(NT4-Pad2)
- added copper zone on F.Cu, net Net-(NT5-Pad2)
- added copper zone on F.Cu, net Net-(NT8-Pad2)
- added copper zone on B.Cu, net V_SUPPLY
Other:
- board size 67 x 90 mm -> 60 x 100 mm
- board text added: "ESC-power-epc v0.1 6/01/22"
- board text added: "JLCJLCJLCJLC"
