File: ESC-power-epc.kicad_sch (KiCad schematic)
At the start: 9 parts, among them J1 GATE, J2 Conn_01x02, J3 Conn_01x04, J4 GATE

Commit message: before changing connector
Parts:
- J1, J4: footprint (none) -> Connector_PinHeader_2.54mm:PinHeader_2x04_P2.54mm_Vertical
- J2: footprint (none) -> Connector_PinHeader_2.54mm:PinHeader_1x02_P2.54mm_Vertical
- J3: footprint (none) -> Connector_PinHeader_2.54mm:PinHeader_2x02_P2.54mm_Vertical
Connections:
- net GND: now also J4.7 (Pin_7), J4.8 (Pin_8)
- net +5V: now reaches J4.1 (Pin_1)
- net +3V3: now reaches J4.2 (Pin_2)
- net GATE/H1: now reaches J1.1 (Pin_1)
- net GATE/H2: now reaches J1.3 (Pin_3)
- net GATE/H3: now reaches J1.4 (Pin_4)
- net GATE/L1: now reaches J1.5 (Pin_5)
- net GATE/L2: now reaches J1.6 (Pin_6)
- net GATE/L3: now reaches J1.7 (Pin_7)
- net MOSFETS/CURR_A renamed CURRENT_A
- net MOSFETS/CURR_B renamed CURRENT_B
- net MOSFETS/CURR_C renamed CURRENT_C
- net MOSFETS/SENSE_A renamed SENSE_A
- net MOSFETS/SENSE_B renamed SENSE_B
- net MOSFETS/SENSE_C renamed SENSE_C
- net MOSFETS/VSA renamed GATE/VSA
- net MOSFETS/VSB renamed GATE/VSB
- net MOSFETS/VSC renamed GATE/VSC
Other:
- removed sheet MOSFETS
- added sheet GaN_A (GaN.kicad_sch)
- added sheet GaN_B (GaN.kicad_sch)
- added sheet GaN_C (GaN.kicad_sch)
- sheet GATE ports: added GH_A, GH_B, GH_C, GL_A, GL_B, GL_C, H1, H2, H3, L1, L2, L3, VSA, VSB, VSC; removed none
- moved on the sheet: H3, H4, H5

Commit message: before meeting
Connections:
- net +12V: now also J4.8 (Pin_8); no longer J1.8 (Pin_8)
- net +3V3: now also J4.1 (Pin_1); no longer J4.2 (Pin_2)
- net +5V: now also J1.7 (Pin_7); no longer J4.1 (Pin_1)
- net GATE/H1: now also J1.4 (Pin_4); no longer J1.1 (Pin_1)
- net GATE/H2: now also J1.2 (Pin_2); no longer J1.3 (Pin_3)
- net GATE/H3: now also J1.1 (Pin_1); no longer J1.4 (Pin_4)
- net GATE/L1: now also J1.8 (Pin_8); no longer J1.5 (Pin_5)
- net GATE/L3: now also J1.5 (Pin_5); no longer J1.7 (Pin_7)
- net GND: now also J1.3 (Pin_3), J4.2 (Pin_2); no longer J1.2 (Pin_2), J4.8 (Pin_8)
- net TEMP_MOSFET: now reaches J4.6 (Pin_6)

Commit message: v0.1
Parts:
- added C35, C61, C67: 10u/100V, Capacitor_SMD:C_2220_5650Metric, symbol Device:C
- added C75: 660u, Capacitor_THT:CP_Radial_D12.5mm_P5.00mm, symbol Device:C_Polarized
- added C76: 2u2, Capacitor_SMD:C_0805_2012Metric, symbol Device:C
- added H10, H11, H6, H7, H8, H9: MountingHole, MountingHole:MountingHole_3.2mm_M3, symbol Mechanical:MountingHole
- added R48: NTC 10k, Resistor_SMD:R_0603_1608Metric, symbol Device:R
- added R49: 10k, Resistor_SMD:R_0805_2012Metric, symbol Device:R
- added TP1, TP2: GND, TestPoint:TestPoint_THTPad_D1.5mm_Drill0.7mm, symbol Connector:TestPoint
Connections:
- net +3V3: now also R48.1
- net GND: now also C35.2, C61.2, C67.2, C75.2, C76.2, R49.2, TP1.1, TP2.1
- net V_SUPPLY: now also C35.1, C61.1, C67.1, C75.1
- net Gate drivers/VSA renamed VSA
- net Gate drivers/VSB renamed VSB
- net Gate drivers/VSC renamed VSC
- net TEMP_MOSFET renamed TEMP_FET
- net TEMP_FET: now also C76.1, R48.2, R49.1
Other:
- sheet GATE renamed Gate drivers
