File: GaN.kicad_sch (KiCad schematic)
At the start: 36 parts, among them Q1 EPC2302, Q4 EPC2302, U3 INA181A2

Commit message: before changing connector
Parts:
- removed R7, R8: 3m, Resistor_SMD:R_0805_2012Metric, symbol Device:R
- added R12, R13: 3m, Froste:0805W, symbol Device:R
- C35: renamed from C?; footprint (none) -> Capacitor_SMD:C_0805_2012Metric
- R25: renamed from R?; footprint (none) -> Resistor_SMD:R_2512_6332Metric
- R5, R6: footprint Resistor_SMD:R_0805_2012Metric -> Froste:0805W; LCSC C500611 -> C2692046
- gave numbers to parts that had none: 3
Connections:
- net GND: now also R12.2, R13.2
- net at NT1.2, Q4.2, Q4.4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: now also R12.1, R13.1
- net CURR_A renamed CURR
- net GH_A renamed GH
- net GL_A renamed GL
- net SENSE_A renamed SENSE
- net VSA renamed VS
Changed lines of the file:
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@@
     )
   )
-  (hierarchical_label "VSA" (shape input) (at 74.93 74.93 180)
+  (hierarchical_label "VS" (shape input) (at 74.93 74.93 180)
     (effects (font (size 1.27 1.27)) (justify right))
   )
-  (hierarchical_label "GH_A" (shape input) (at 144.78 67.31 180)
+  (hierarchical_label "GH" (shape input) (at 144.78 67.31 180)
     (effects (font (size 1.27 1.27)) (justify right))
   )
-  (hierarchical_label "VSA" (shape input) (at 40.64 168.91 180)
+  (hierarchical_label "VS" (shape input) (at 40.64 168.91 180)
     (effects (font (size 1.27 1.27)) (justify right))
   )
-  (hierarchical_label "SENSE_A" (shape input) (at 58.42 168.91 0)
+  (hierarchical_label "SENSE" (shape input) (at 58.42 168.91 0)
     (effects (font (size 1.27 1.27)) (justify left))
   )
-  (hierarchical_label "GL_A" (shape input) (at 143.51 116.84 180)
+  (hierarchical_label "GL" (shape input) (at 143.51 116.84 180)
     (effects (font (size 1.27 1.27)) (justify right))
   )
-  (hierarchical_label "CURR_A" (shape input) (at 154.94 173.99 0)
+  (hierarchical_label "CURR" (shape input) (at 154.94 173.99 0)
     (effects (font (size 1.27 1.27)) (justify left))
   )
   (symbol (lib_id "Device:R") (at 90.17 74.93 270) (unit 1)
     (in_bom yes) (on_board yes) (fields_autoplaced)
-    (property "Reference" "R?" (id 0) (at 90.17 68.58 90))
+    (property "Reference" "R25" (id 0) (at 90.17 68.58 90))
     (property "Value" "R" (id 1) (at 90.17 71.12 90))
-    (property "Footprint" "" (id 2) (at 90.17 73.152 90)
+    (property "Footprint" "Resistor_SMD:R_2512_6332Metric" (id 2) (at 90.17 73.152 90)
       (effects (font (size 1.27 1.27)) hide)
     )
@@
       (effects (font (size 1.27 1.27)) (justify right))
     )
-    (property "Footprint" "Resistor_SMD:R_0805_2012Metric" (id 2) (at 138.938 127 90)
+    (property "Footprint" "Froste:0805W" (id 2) (at 138.938 127 90)
       (effects (font (size 1.27 1.27)) hide)
     )
@@
       (effects (font (size 1.27 1.27)) hide)
     )
-    (property "LCSC" " C500611" (id 4) (at 137.16 127 0)
+    (property "LCSC" "C2692046" (id 4) (at 137.16 127 0)
       (effects (font (size 1.27 1.27)) hide)
     )
@@
   (symbol (lib_id "Device:C") (at 100.33 102.87 0) (unit 1)
     (in_bom yes) (on_board yes) (fields_autoplaced)
-    (property "Reference" "C?" (id 0) (at 104.14 101.5999 0)
+    (property "Reference" "C35" (id 0) (at 104.14 101.5999 0)
       (effects (font (size 1.27 1.27)) (justify left))
     )
@@
       (effects (font (size 1.27 1.27)) (justify left))
     )
-    (property "Footprint" "" (id 2) (at 101.2952 106.68 0)
+    (property "Footprint" "Capacitor_SMD:C_0805_2012Metric" (id 2) (at 101.2952 106.68 0)
       (effects (font (size 1.27 1.27)) hide)
     )
@@
     (pin "2")
   )
-  (symbol (lib_id "Device:R") (at 146.05 127 0) (mirror y) (unit 1)
-    (in_bom yes) (on_board yes) (fields_autoplaced)
-    (property "Reference" "R8" (id 0) (at 148.59 125.7299 0)
-      (effects (font (size 1.27 1.27)) (justify right))
-    )
-    (property "Value" "3m" (id 1) (at 148.59 128.2699 0)
-      (effects (font (size 1.27 1.27)) (justify right))
-    )
-    (property "Footprint" "Resistor_SMD:R_0805_2012Metric" (id 2) (at 147.828 127 90)
-      (effects (font (size 1.27 1.27)) hide)
-    )
-    (property "Datasheet" "~" (id 3) (at 146.05 127 0)
-      (effects (font (size 1.27 1.27)) hide)
-    )
-    (property "LCSC" " C500611" (id 4) (at 146.05 127 0)
-      (effects (font (size 1.27 1.27)) hide)
-    )
-    (pin "1")
-    (pin "2")
-  )
   (symbol (lib_id "Device:C") (at 224.79 30.48 0) (unit 1)
     (in_bom yes) (on_board yes)
@@
   (symbol (lib_id "Amplifier_Current:INA240A1D") (at 90.17 99.06 270) (unit 1)
     (in_bom yes) (on_board yes) (fields_autoplaced)
-    (property "Reference" "U?" (id 0) (at 94.869 110.49 0))
+    (property "Reference" "U7" (id 0) (at 94.869 110.49 0))
     (property "Value" "INA240A1D" (id 1) (at 92.329 110.49 0))
     (property "Footprint" "Package_SO:SOIC-8_3.9x4.9mm_P1.27mm" (id 2) (at 73.66 99.06 0)
@@
   (symbol (lib_id "Device:NetTie_2") (at 96.52 80.01 90) (unit 1)
     (in_bom yes) (on_board yes)
-    (property "Reference" "NT?" (id 0) (at 97.79 80.01 0))
+    (property "Reference" "NT8" (id 0) (at 97.79 80.01 0))
     (property "Value" "NetTie_2" (id 1) (at 93.98 80.01 0)
       (effects (font (size 1.27 1.27)) hide)
@@
   (symbol (lib_id "power:GND") (at 100.33 109.22 0) (unit 1)
     (in_bom yes) (on_board yes) (fields_autoplaced)
-    (property "Reference" "#PWR?" (id 0) (at 100.33 115.57 0)
+    (property "Reference" "#PWR0132" (id 0) (at 100.33 115.57 0)
       (effects (font (size 1.27 1.27)) hide)
     )
@@
   (symbol (lib_id "power:+3V3") (at 100.33 92.71 0) (unit 1)
     (in_bom yes) (on_board yes)
-    (property "Reference" "#PWR?" (id 0) (at 100.33 96.52 0)
+    (property "Reference" "#PWR0131" (id 0) (at 100.33 96.52 0)
       (effects (font (size 1.27 1.27)) hide)
     )
@@
   (symbol (lib_id "Device:R") (at 154.94 127 0) (mirror y) (unit 1)
     (in_bom yes) (on_board yes) (fields_autoplaced)
-    (property "Reference" "R7" (id 0) (at 157.48 125.7299 0)
+    (property "Reference" "R13" (id 0) (at 157.48 125.7299 0)
       (effects (font (size 1.27 1.27)) (justify right))
     )
@@
       (effects (font (size 1.27 1.27)) (justify right))
     )
-    (property "Footprint" "Resistor_SMD:R_0805_2012Metric" (id 2) (at 156.718 127 90)
+    (property "Footprint" "Froste:0805W" (id 2) (at 156.718 127 90)
       (effects (font (size 1.27 1.27)) hide)
     )
@@
       (effects (font (size 1.27 1.27)) hide)
     )
-    (property "LCSC" " C500611" (id 4) (at 154.94 127 0)
+    (property "LCSC" "C2692046" (id 4) (at 154.94 127 0)
       (effects (font (size 1.27 1.27)) hide)
     )
@@
     (pin "2")
   )
+  (symbol (lib_id "Device:R") (at 146.05 127 0) (mirror y) (unit 1)
+    (in_bom yes) (on_board yes) (fields_autoplaced)
+    (property "Reference" "R12" (id 0) (at 148.59 125.7299 0)
+      (effects (font (size 1.27 1.27)) (justify right))
+    )
+    (property "Value" "3m" (id 1) (at 148.59 128.2699 0)
+      (effects (font (size 1.27 1.27)) (justify right))
+    )
+    (property "Footprint" "Froste:0805W" (id 2) (at 147.828 127 90)
+      (effects (font (size 1.27 1.27)) hide)
+    )
+    (property "Datasheet" "~" (id 3) (at 146.05 127 0)
+      (effects (font (size 1.27 1.27)) hide)
+    )
+    (property "LCSC" "C2692046" (id 4) (at 146.05 127 0)
+      (effects (font (size 1.27 1.27)) hide)
+    )
+    (pin "1")
+    (pin "2")
+  )
   (symbol (lib_id "power:GND") (at 90.17 109.22 0) (unit 1)
     (in_bom yes) (on_board yes) (fields_autoplaced)
-    (property "Reference" "#PWR?" (id 0) (at 90.17 115.57 0)
+    (property "Reference" "#PWR0133" (id 0) (at 90.17 115.57 0)
       (effects (font (size 1.27 1.27)) hide)
     )
@@
       (effects (font (size 1.27 1.27)) (justify right))
     )
-    (property "Footprint" "Resistor_SMD:R_0805_2012Metric" (id 2) (at 130.048 127 90)
+    (property "Footprint" "Froste:0805W" (id 2) (at 130.048 127 90)
       (effects (font (size 1.27 1.27)) hide)
     )
@@
       (effects (font (size 1.27 1.27)) hide)
     )
-    (property "LCSC" " C500611" (id 4) (at 128.27 127 0)
+    (property "LCSC" "C2692046" (id 4) (at 128.27 127 0)
       (effects (font (size 1.27 1.27)) hide)
     )
@@
   (symbol (lib_id "Device:NetTie_2") (at 83.82 80.01 270) (unit 1)
     (in_bom yes) (on_board yes)
-    (property "Reference" "NT?" (id 0) (at 82.55 80.01 0))
+    (property "Reference" "NT7" (id 0) (at 82.55 80.01 0))
     (property "Value" "NetTie_2" (id 1) (at 86.36 80.01 0)
       (effects (font (size 1.27 1.27)) hide)

Commit message: before meeting
Parts:
- renumbered R12 to R7, R13 to R8
Other:
- moved on the sheet: NT8
Changed lines of the file:
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@@
     (pin "2")
   )
-  (symbol (lib_id "Device:NetTie_2") (at 96.52 80.01 90) (unit 1)
-    (in_bom yes) (on_board yes)
-    (property "Reference" "NT8" (id 0) (at 97.79 80.01 0))
-    (property "Value" "NetTie_2" (id 1) (at 93.98 80.01 0)
+  (symbol (lib_id "Device:NetTie_2") (at 96.52 80.01 270) (mirror x) (unit 1)
+    (in_bom yes) (on_board yes)
+    (property "Reference" "NT8" (id 0) (at 95.25 80.01 0))
+    (property "Value" "NetTie_2" (id 1) (at 99.06 80.01 0)
       (effects (font (size 1.27 1.27)) hide)
     )
@@
   (symbol (lib_id "Device:R") (at 154.94 127 0) (mirror y) (unit 1)
     (in_bom yes) (on_board yes) (fields_autoplaced)
-    (property "Reference" "R13" (id 0) (at 157.48 125.7299 0)
+    (property "Reference" "R8" (id 0) (at 157.48 125.7299 0)
       (effects (font (size 1.27 1.27)) (justify right))
     )
@@
   (symbol (lib_id "Device:R") (at 146.05 127 0) (mirror y) (unit 1)
     (in_bom yes) (on_board yes) (fields_autoplaced)
-    (property "Reference" "R12" (id 0) (at 148.59 125.7299 0)
+    (property "Reference" "R7" (id 0) (at 148.59 125.7299 0)
       (effects (font (size 1.27 1.27)) (justify right))
     )

Commit message: v0.1
Parts:
- removed C35: 1u, Capacitor_SMD:C_0805_2012Metric, symbol Device:C
- removed R25: R, Resistor_SMD:R_2512_6332Metric, symbol Device:R
- removed U7: INA240A1D, Package_SO:SOIC-8_3.9x4.9mm_P1.27mm, symbol Amplifier_Current:INA240A1D
- added C78: 2u2, Capacitor_SMD:C_0805_2012Metric, symbol Device:C
- added JP2: Jumper_3_Bridged12, Jumper:SolderJumper-3_P1.3mm_Open_RoundedPad1.0x1.5mm, symbol Jumper:Jumper_3_Bridged12
- added R52: 1m, Resistor_SMD:R_2512_6332Metric, symbol Device:R
- added U7: AD8418, Package_SO:MSOP-8_3x3mm_P0.65mm, symbol Amplifier_Current:AD8418
- C38, C39, C40, C41, C42, C43, C44, C45: LCSC C412614 -> C2981733
- NT1, NT2: footprint NetTie:NetTie-2_SMD_Pad0.5mm -> Froste:NetTie-2_SMD_Pad0.26mm
- R5, R6, R7, R8: value 3m -> 2m; LCSC C2692046 -> C2692045
Connections:
- net +3V3: now also C78.1, U7.6 (VS), U7.7 (REF1)
- net CURR: now also JP2.2 (C); no longer C16.1, R26.2
- net GND: now also C78.2, U7.2 (GND), U7.3 (REF2)
- net VS: now also NT7.2, R52.1; no longer NT7.1
- net at NT8.2, Q1.2, Q1.4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: now also R52.2
- net IN+: now reaches NT8.1
- net IN+: now also U7.8 (IN+)
- net +1V5 renamed 1V65
- net SA_N renamed S_N
- net SA_P renamed S_P
- new net CUR_SHUNT_LOW: C16.1, JP2.3 (B), R26.2
- new net CUR_SHUNT_PHASE: JP2.1 (A), U7.5 (OUT)
- new net IN-: NT7.1, U7.1 (IN-)
